Commit message: ros2 controls added

File: src/sort_robo_description/urdf/gazebo.xacro (robot description, xacro)
@@ -1,91 +1,24 @@
 <?xml version="1.0"?>
 <robot xmlns:xacro="http://www.ros.org/wiki/xacro" name="panda">
-  <xacro:property name="PI" value="3.14159265359" />
-  <ros2_control name="RobotSystem" type="system">
-    <!-- ros2_control Gazebo -->
-    <!-- ROS 2 Humble -->
+  <!-- ROS 2 Control -->
+  <!-- ROS 2 Humble -->
+  <gazebo>
     <xacro:if value="$(arg is_ignition)">
-      <hardware>
-        <plugin>ign_ros2_control/IgnitionSystem</plugin>
-      </hardware>
+      <plugin filename="ign_ros2_control-system" name="ign_ros2_control::IgnitionROS2ControlPlugin">
+        <parameters>$(find sort_robo_controller)/config/controllers.yaml</parameters>
+      </plugin>
+      <plugin filename="ignition-gazebo-sensors-system" name="ignition::gazebo::systems::Sensors">
+        <render_engine>ogre2</render_engine>
+      </plugin>
     </xacro:if>
     <!-- ROS 2 Iron or above -->
     <xacro:unless value="$(arg is_ignition)">
-      <hardware>
-        <plugin>gz_ros2_control/GazeboSimSystem</plugin>
-      </hardware>
+      <plugin filename="gz_ros2_control-system" name="gz_ros2_control::GazeboSimROS2ControlPlugin">
+        <parameters>$(find sort_robo_controller)/config/controllers.yaml</parameters>
+      </plugin>
+      <plugin filename="gz-sim-sensors-system" name="gz::sim::systems::Sensors">
+        <render_engine>ogre2</render_engine>
+      </plugin>
     </xacro:unless>
-    <!-- Joint 1 -->
-    <joint name="panda_joint1">
-      <command_interface name="position">
-        <param name="min">-2.9671</param>
-        <param name="max">2.9671</param>
-      </command_interface>
-      <state_interface name="position"/>
-    </joint>
-    <!-- Joint 2 -->
-    <joint name="panda_joint2">
-      <command_interface name="position">
-        <param name="min">-1.8326</param>
-        <param name="max">1.8326</param>
-      </command_interface>
-      <state_interface name="position"/>
-    </joint>
-    <!-- Joint 3 -->
-    <joint name="panda_joint3">
-      <command_interface name="position">
-        <param name="min">-2.9671</param>
-        <param name="max">2.9671</param>
-      </command_interface>
-      <state_interface name="position"/>
-    </joint>
-    <!-- Joint 4 -->
-    <joint name="panda_joint4">
-      <command_interface name="position">
-        <param name="min">-3.1416</param>
-        <param name="max">0.0</param>
-      </command_interface>
-      <state_interface name="position"/>
-    </joint>
-    <!-- Joint 5 -->
-    <joint name="panda_joint5">
-      <command_interface name="position">
-        <param name="min">-2.9671</param>
-        <param name="max">2.9671</param>
-      </command_interface>
-      <state_interface name="position"/>
-    </joint>
-    <!-- Joint 6 -->
-    <joint name="panda_joint6">
-      <command_interface name="position">
-        <param name="min">-0.0873</param>
-        <param name="max">3.8223</param>
-      </command_interface>
-      <state_interface name="position"/>
-    </joint>
-    <!-- Joint 7 -->
-    <joint name="panda_joint7">
-      <command_interface name="position">
-        <param name="min">-2.9671</param>
-        <param name="max">2.9671</param>
-      </command_interface>
-      <state_interface name="position"/>
-    </joint>
-    <!-- Gripper Finger Joint 1 -->
-    <joint name="panda_finger_joint1">
-      <command_interface name="position">
-        <param name="min">0.0</param>
-        <param name="max">0.04</param>
-      </command_interface>
-      <state_interface name="position"/>
-    </joint>
-    <!-- Gripper Finger Joint 2 (Mimics Joint 1) -->
-    <joint name="panda_finger_joint2">
-      <command_interface name="position">
-        <param name="min">0.0</param>
-        <param name="max">0.04</param>
-      </command_interface>
-      <state_interface name="position"/>
-    </joint>
-  </ros2_control>
+  </gazebo>
 </robot>

File: src/sort_robo_description/urdf/ros2Control.xacro (robot description, xacro)
@@ -1,24 +1,91 @@
 <?xml version="1.0"?>
 <robot xmlns:xacro="http://www.ros.org/wiki/xacro" name="panda">
-  <!-- ROS 2 Control -->
-  <!-- ROS 2 Humble -->
-  <gazebo>
+  <xacro:property name="PI" value="3.14159265359" />
+  <ros2_control name="RobotSystem" type="system">
+    <!-- ros2_control Gazebo -->
+    <!-- ROS 2 Humble -->
     <xacro:if value="$(arg is_ignition)">
-      <plugin filename="ign_ros2_control-system" name="ign_ros2_control::IgnitionROS2ControlPlugin">
-        <parameters>$(find sort_robo_description)/config/controllers.yaml</parameters>
-      </plugin>
-      <plugin filename="ignition-gazebo-sensors-system" name="ignition::gazebo::systems::Sensors">
-        <render_engine>ogre2</render_engine>
-      </plugin>
+      <hardware>
+        <plugin>ign_ros2_control/IgnitionSystem</plugin>
+      </hardware>
     </xacro:if>
     <!-- ROS 2 Iron or above -->
     <xacro:unless value="$(arg is_ignition)">
-      <plugin filename="gz_ros2_control-system" name="gz_ros2_control::GazeboSimROS2ControlPlugin">
-        <parameters>$(find sort_robo_description)/config/controllers.yaml</parameters>
-      </plugin>
-      <plugin filename="gz-sim-sensors-system" name="gz::sim::systems::Sensors">
-        <render_engine>ogre2</render_engine>
-      </plugin>
+      <hardware>
+        <plugin>gz_ros2_control/GazeboSimSystem</plugin>
+      </hardware>
     </xacro:unless>
-  </gazebo>
+    <!-- Joint 1 -->
+    <joint name="panda_joint1">
+      <command_interface name="position">
+        <param name="min">-2.9671</param>
+        <param name="max">2.9671</param>
+      </command_interface>
+      <state_interface name="position"/>
+    </joint>
+    <!-- Joint 2 -->
+    <joint name="panda_joint2">
+      <command_interface name="position">
+        <param name="min">-1.8326</param>
+        <param name="max">1.8326</param>
+      </command_interface>
+      <state_interface name="position"/>
+    </joint>
+    <!-- Joint 3 -->
+    <joint name="panda_joint3">
+      <command_interface name="position">
+        <param name="min">-2.9671</param>
+        <param name="max">2.9671</param>
+      </command_interface>
+      <state_interface name="position"/>
+    </joint>
+    <!-- Joint 4 -->
+    <joint name="panda_joint4">
+      <command_interface name="position">
+        <param name="min">-3.1416</param>
+        <param name="max">0.0</param>
+      </command_interface>
+      <state_interface name="position"/>
+    </joint>
+    <!-- Joint 5 -->
+    <joint name="panda_joint5">
+      <command_interface name="position">
+        <param name="min">-2.9671</param>
+        <param name="max">2.9671</param>
+      </command_interface>
+      <state_interface name="position"/>
+    </joint>
+    <!-- Joint 6 -->
+    <joint name="panda_joint6">
+      <command_interface name="position">
+        <param name="min">-0.0873</param>
+        <param name="max">3.8223</param>
+      </command_interface>
+      <state_interface name="position"/>
+    </joint>
+    <!-- Joint 7 -->
+    <joint name="panda_joint7">
+      <command_interface name="position">
+        <param name="min">-2.9671</param>
+        <param name="max">2.9671</param>
+      </command_interface>
+      <state_interface name="position"/>
+    </joint>
+    <!-- Gripper Finger Joint 1 -->
+    <joint name="panda_finger_joint1">
+      <command_interface name="position">
+        <param name="min">0.0</param>
+        <param name="max">0.04</param>
+      </command_interface>
+      <state_interface name="position"/>
+    </joint>
+    <!-- Gripper Finger Joint 2 (Mimics Joint 1) -->
+    <joint name="panda_finger_joint2">
+      <command_interface name="position">
+        <param name="min">0.0</param>
+        <param name="max">0.04</param>
+      </command_interface>
+      <state_interface name="position"/>
+    </joint>
+  </ros2_control>
 </robot>
