Commit message: updates for the arm

File: src/sort_robo_description/urdf/sensors.xacro (robot description, xacro)
@@ -12,5 +12,7 @@
                 <box size="0.1 0.1 0.05"/>
             </geometry>
-            <material name="red"/>
+            <material name="camera_housing">
+                <color rgba="0.3 0.3 0.3 1.0"/>
+            </material>
         </visual>
         <collision>
@@ -19,9 +21,8 @@
                 <box size="0.1 0.1 0.05"/>
             </geometry>
-            <material name="red"/>
         </collision>
     </link>
     <joint name="camera_joint" type="fixed">
-        <origin xyz="0.6 0 1.0" rpy="0.0 0.0 0.0"/>
+        <origin xyz="0.6 0.6 1.1" rpy="0.0 0.0 0.0"/>
         <parent link="panda_link0"/>
         <child link="camera_link"/>
@@ -34,4 +35,5 @@
     </joint>
     <gazebo reference="camera_link">
+        <material>Gazebo/Grey</material>
         <sensor name="camera" type="camera">
             <pose>0 0 0 0 1.57 0</pose>
@@ -55,4 +57,57 @@
             </camera>
         </sensor>
-  </gazebo>
+        <!-- Depth camera — same pose/FOV as RGB, replaces hardcoded depth assumption -->
+        <sensor name="depth_camera" type="depth_camera">
+            <pose>0 0 0 0 1.57 0</pose>
+            <always_on>true</always_on>
+            <update_rate>10</update_rate>
+            <topic>camera/depth/image_raw</topic>
+            <gz_frame_id>camera_link_optical</gz_frame_id>
+            <camera>
+                <horizontal_fov>1.0</horizontal_fov>
+                <image>
+                    <width>640</width>
+                    <height>320</height>
+                    <format>R_FLOAT32</format>
+                </image>
+                <clip>
+                    <near>0.05</near>
+                    <far>8.0</far>
+                </clip>
+            </camera>
+        </sensor>
+    </gazebo>
+    <!-- IMU link — co-located with camera, foundation for camera-IMU (VIO) fusion -->
+    <link name="imu_link">
+        <inertial>
+            <origin xyz="0 0 0" rpy="0 0 0"/>
+            <mass value="0.01"/>
+            <inertia ixx="1e-5" ixy="0" ixz="0" iyy="1e-5" iyz="0" izz="1e-5"/>
+        </inertial>
+    </link>
+    <joint name="imu_joint" type="fixed">
+        <parent link="camera_link"/>
+        <child link="imu_link"/>
+        <origin xyz="0 0 0" rpy="0 0 0"/>
+    </joint>
+    <gazebo reference="imu_link">
+        <sensor name="imu_sensor" type="imu">
+            <always_on>true</always_on>
+            <update_rate>100</update_rate>
+            <topic>imu/data</topic>
+            <gz_frame_id>imu_link</gz_frame_id>
+            <imu>
+                <angular_velocity>
+                    <x><noise type="gaussian"><mean>0.0</mean><stddev>2e-4</stddev></noise></x>
+                    <y><noise type="gaussian"><mean>0.0</mean><stddev>2e-4</stddev></noise></y>
+                    <z><noise type="gaussian"><mean>0.0</mean><stddev>2e-4</stddev></noise></z>
+                </angular_velocity>
+                <linear_acceleration>
+                    <x><noise type="gaussian"><mean>0.0</mean><stddev>1.7e-2</stddev></noise></x>
+                    <y><noise type="gaussian"><mean>0.0</mean><stddev>1.7e-2</stddev></noise></y>
+                    <z><noise type="gaussian"><mean>0.0</mean><stddev>1.7e-2</stddev></noise></z>
+                </linear_acceleration>
+            </imu>
+        </sensor>
+    </gazebo>
 </robot>

Commit message: dockerized everything

File: src/sort_robo_description/urdf/sensors.xacro (robot description, xacro)
@@ -24,5 +24,5 @@
     </link>
     <joint name="camera_joint" type="fixed">
-        <origin xyz="0.6 0.6 1.1" rpy="0.0 0.0 0.0"/>
+        <origin xyz="0.6 0 1.0" rpy="0.0 0.0 0.0"/>
         <parent link="panda_link0"/>
         <child link="camera_link"/>
